File: kicad_source/DronecodeCANAdapter.sch (KiCad schematic (older format))
At the start: 31 parts, among them CN1 RASPI-IO, CN2 691322310004, CN3 GH_SM04B-GHS-TB, CN4 GH_SM04B-GHS-TB, SW1 JS202011JCQN, U1 MCP2518FD, U2 TCAN332GDR, Y1 RH100-20.000-20-3030-TR

Commit message: updated schematic and layout
Parts:
- removed C1: 100nF, capacitors:C_0603, symbol devices:C_0603
- removed C2, C3: 22pF, capacitors:C_0603, symbol devices:C_0603
- removed CN1: RASPI-IO, MODULE_compute:RASPI_ZERO_HAT_EDGE, symbol MODULE_compute:RASPI-IO
- removed L2: Label, labels:generationmake_logo, symbol devices:Label
- removed R1, R8: 0R, resistors:R_0603, symbol devices:R_0603
- removed R2, R6, R7, R9: DNI, resistors:R_0603, symbol devices:R_0603
- removed R3, R5: 10k, resistors:R_0603, symbol devices:R_0603
- removed SW1: JS202011JCQN, mechanical-switches:CK_JS202011JCQN, symbol devices:SWITCH_SMALL
- removed U1: MCP2518FD, SOIC:SOIC-14_3.9x8.7mm_Pitch1.27mm, symbol IC_transceiver_can:MCP2517FD
- removed Y1: RH100-20.000-20-3030-TR, crystals:Crystal_SMD_3.2x2.5mm_4Pad, symbol devices:Crystal_SMD_4Pad
- added CN1: CONN_01X05, pin_headers:Pin_Header_Straight_1x05, symbol mechanical-connectors:CONN_01X05
- added MECH1, MECH2: MHP_3.2_5.0, MECH_mounting_holes:MHP_3.2_5.0, symbol MECH_mounting-holes:MHP_3.2_5.0
- L1: footprint labels:generationmake_small_solder -> labels:generationmake_small_silk
- R4: value 120R -> DNI
- renumbered C4 to C1, D2 to D1, D3 to D2, D4 to D3, D1 to D4, R10 to R1, R11 to R2, R12 to R3, U2 to U1
Connections:
- net labels removed: I2C_SCL, I2C_SDA, INTERRUPT_12, INTERRUPT_23, INTERRUPT_24, INTERRUPT_25, MCP2517_CS, MCP2517_INT, OSC1, OSC2, SERIAL_RX, SERIAL_TX, SPI_CE0, SPI_CE1, SPI_CLK, SPI_MISO, SPI_MOSI
- wire segments 135 -> 59
- no-connect marks 21 -> 4
Other:
- note removed: "20 MHz"
